File: asd1025-relayed-v1/asd1025-relayed-v1.kicad_pcb (KiCad board)
At the start: 2 copper layers, 76.2 x 57.2 mm, 36 parts, among them J1 Conn_01x09_Female, J10 Conn_01x01_Female, J11 Conn_01x01_Female, J12 Conn_01x01_Female, J13 Conn_01x01_Female, J14 Conn_01x01_Female, J15 Conn_01x01_Female, J16 Conn_01x01_Female, J17 Conn_01x01_Female, J18 Conn_01x01_Female, J19 Conn_01x01_Female, J2 Conn_01x01_Female, J20 Conn_01x01_Female, J21 Conn_01x01_Female, J22 Conn_01x01_Female, J3 Conn_01x01_Female, J4 Conn_01x01_Female, J5 Conn_01x01_Female, J6 Conn_01x01_Female, J7 Conn_01x01_Female, J8 Conn_01x01_Female, J9 Conn_01x01_Female, K1 EC2-4.5NU, K2 EC2-4.5NU, K3 EC2-4.5NU, K4 EC2-4.5NU, K5 EC2-4.5NU, K6 EC2-4.5NU, Q1 BC547, U1 SA555P, U2 74HC02, U3 4017, U4 ULN2004A

Commit message: fix v1: relays would switch by passing current through base-emittor-resistors in darlington array even if main transistor Q1 is off
Parts:
- Q1: value BC547 -> BC557; footprint Package_TO_SOT_THT:TO-92L_Inline_Wide -> Package_TO_SOT_THT:TO-92_Inline_Wide
- U2: value 74HC02 -> 74HC00
- U4: value ULN2004A -> ULN2003A
- moved Q1 39.8 mm to (61.0, 134.6)
- moved U2 17.0 mm to (66.0, 165.1), turned to 180 degrees
- moved R2 10.5 mm to (71.1, 152.4), turned to 90 degrees
Connections:
- J1 pad 9: Net-(J1-Pad9) -> Net-(U2-Pad9)
- K1 pad 1: +5V -> Net-(K1-Pad1)
- K2 pad 1: +5V -> Net-(K1-Pad1)
- K3 pad 1: +5V -> Net-(K1-Pad1)
- K4 pad 1: +5V -> Net-(K1-Pad1)
- K5 pad 1: +5V -> Net-(K1-Pad1)
- K6 pad 1: +5V -> Net-(K1-Pad1)
- Q1 pad 1: Net-(Q1-Pad1) -> Net-(K1-Pad1)
- Q1 pad 3: GNDREF -> +5V
- U1 pad 4: +5V -> Net-(R2-Pad1)
- U2 pad 1: Net-(R2-Pad1) -> Net-(J1-Pad1)
- U2 pad 12: Net-(J1-Pad1) -> Net-(U2-Pad9)
- U2 pad 13: Net-(U2-Pad13) -> Net-(J1-Pad1)
- U2 pad 2: Net-(U2-Pad13) -> Net-(U2-Pad10)
- U2 pad 5: Net-(U2-Pad10) -> Net-(U2-Pad8)
- U2 pad 6: Net-(J1-Pad9) -> Net-(R2-Pad1)
- U2 pad 8: Net-(J1-Pad9) -> Net-(U2-Pad8)
- U2 pad 9: Net-(J1-Pad1) -> Net-(U2-Pad9)
- U3 pad 13: Net-(R2-Pad1) -> GNDREF
- U4 pad 8: Net-(Q1-Pad1) -> GNDREF
- U4 pad 9: +5V -> Net-(K1-Pad1)
Routing:
- net +5V: track 191.9 -> 106.7 mm
- net Net-(K1-Pad1): track 0.00 -> 79.8 mm
- net Net-(R2-Pad1): track 70.4 -> 29.6 mm
- net GNDREF: track 65.6 -> 95.8 mm
- net Net-(U2-Pad9): track 0.00 -> 25.0 mm
- net Net-(J1-Pad9): track 19.9 -> 0.00 mm
- net Net-(U2-Pad8): track 0.00 -> 9.72 mm
- net Net-(U2-Pad13): track 7.62 -> 0.00 mm
- net Net-(Q1-Pad2): track 5.08 -> 12.3 mm
- net Net-(Q1-Pad1): track 6.13 -> 0.00 mm
- net Net-(J1-Pad1): track 20.9 -> 18.4 mm
- net Net-(U2-Pad10): track 10.2 -> 12.3 mm
Other:
- board text added: "Pioneer A-502R Relay Input Selection replaces switch motor v1 / 2023-03"
- board text removed: "Pioneer A-502R Relay Input Selection replaces switch motor v1 / 2023-02"
